Commit message: Add coalision tag

File: urdf/robot_model.urdf (robot description, URDF)
Before this commit: robot robot_model, 2 links, 1 joints
Links:
- link base_link: mass None -> 10; geometry collision cylinder length=0.6 radius=0.2; visual cylinder length=0.6 radius=0.2
- link right_leg: mass None -> 10; geometry collision box size=0.6 0.1 0.2; visual box size=0.6 0.1 0.2

Commit message: Add gazebo control

File: urdf/robot_model.urdf (robot description, URDF)
Before this commit: robot robot_model, 2 links, 1 joints
Links:
- removed link right_leg
- added link back_left_wheel, mass 10; collision cylinder length=0.6 radius=0.2; visual cylinder length=0.6 radius=0.2
- added link back_right_wheel, mass 10; collision cylinder length=0.6 radius=0.2; visual cylinder length=0.6 radius=0.2
- added link front_left_wheel, mass 10; collision cylinder length=0.6 radius=0.2; visual cylinder length=0.6 radius=0.2
- added link front_right_wheel, mass 10; collision cylinder length=0.6 radius=0.2; visual cylinder length=0.6 radius=0.2
- link base_link: geometry collision box size=0.6 0.1 0.2; visual box size=0.6 0.1 0.2
Joints:
- added joint base_to_left_leg: type continuous, parent base_link, child back_left_wheel, origin xyz=0 -0.22 0.25
- added joint front_left_s: type continuous, parent base_link, child front_left_wheel, origin xyz=0 -0.22 0.25
- added joint front_right_s: type continuous, parent base_link, child front_right_wheel, origin xyz=0 -0.22 0.25
- joint base_to_right_leg: child right_leg -> back_right_wheel; limit lower=-0.38 upper=0 effort=1000.0 velocity=0.5 -> (none); type revolute -> continuous
